File: sc_karltron/sc_karltron.kicad_sch (KiCad schematic)
At the start: 6 parts, among them J1 Conn_01x02, J2 Conn_01x02

Commit message: basic components
Parts:
- added C1, C2, C3, C4, C5: C, Capacitor_THT:C_Disc_D5.0mm_W2.5mm_P5.00mm, symbol Device:C
- added C6: C_Polarized, Capacitor_THT:CP_Radial_D5.0mm_P2.50mm, symbol Device:C_Polarized
- added R1, R10, R13, R15, R17, R19, R2, R3, R6: 100K, Resistor_THT:R_Axial_DIN0207_L6.3mm_D2.5mm_P10.16mm_Horizontal, symbol Device:R
- added R11, R4, R8: LDR, Resistor_THT:R_Axial_DIN0207_L6.3mm_D2.5mm_P10.16mm_Horizontal, symbol Device:R
- added R12, R14, R5, R7, R9: 10K, Resistor_THT:R_Axial_DIN0207_L6.3mm_D2.5mm_P10.16mm_Horizontal, symbol Device:R
- added R16, R18, R20: 1M, Resistor_THT:R_Axial_DIN0207_L6.3mm_D2.5mm_P10.16mm_Horizontal, symbol Device:R
- added RV1, RV2, RV3, RV4: B100K, Potentiometer_THT:Potentiometer_ACP_CA9-V10_Vertical, symbol Device:R_Potentiometer
- added U1, U2: TL074, Package_DIP:DIP-14_W7.62mm, symbol Amplifier_Operational:TL074

Commit message: working too
Parts:
- added D1, D2, D3: LED, LED_THT:LED_D5.0mm_Horizontal_O3.81mm_Z3.0mm, symbol Device:LED
- added J3: In1, Connector_PinHeader_2.54mm:PinHeader_1x02_P2.54mm_Vertical, symbol Connector:AudioJack2
- added J4: Out1, Connector_PinHeader_2.54mm:PinHeader_1x02_P2.54mm_Vertical, symbol Connector:AudioJack2
- added J5: Out2, Connector_PinHeader_2.54mm:PinHeader_1x02_P2.54mm_Vertical, symbol Connector:AudioJack2
- added J6: In2, Connector_PinHeader_2.54mm:PinHeader_1x02_P2.54mm_Vertical, symbol Connector:AudioJack2
- added J7: Out3, Connector_PinHeader_2.54mm:PinHeader_1x02_P2.54mm_Vertical, symbol Connector:AudioJack2
- added J8: Out4, Connector_PinHeader_2.54mm:PinHeader_1x02_P2.54mm_Vertical, symbol Connector:AudioJack2
- added J9: In3, Connector_PinHeader_2.54mm:PinHeader_1x02_P2.54mm_Vertical, symbol Connector:AudioJack2
- added R21, R22, R23: RLED, Resistor_THT:R_Axial_DIN0207_L6.3mm_D2.5mm_P10.16mm_Horizontal, symbol Device:R
- added RV5, RV6, RV7, RV8: B100K, Potentiometer_THT:Potentiometer_Alpha_RD901F-40-00D_Single_Vertical, symbol Device:R_Potentiometer
- C4, C5: value C -> 100nF
- C6: value C_Polarized -> 10uF
- RV1, RV2, RV3, RV4: footprint Potentiometer_THT:Potentiometer_ACP_CA9-V10_Vertical -> Potentiometer_THT:Potentiometer_ACP_CA9-H5_Horizontal
Connections:
- net +9V: now also C4.1, C5.1, C6.1, R7.1, U1.4 (V+), U2.4 (V+)
- net GND: now also C4.2, C5.2, C6.2, R14.2, U1.11 (V-), U2.11 (V-), J3.S, J4.S, J5.S, J6.S, J7.S, J8.S, J9.S, R21.1, R22.1, R23.1
- net Out2: now reaches R2.1
- net Out2: now also J5.T
- net at R2.2: now also R1.2, R3.2, RV4.2, RV4.3, U2.6 (-), RV8.2, RV8.3
- net VMID: now reaches R14.1
- net VMID: now also R7.2, U2.12 (+)
- net Out4: now reaches RV4.1
- net Out4: now also U2.7, J8.T, RV8.1
- net Out3: now reaches R3.1
- net Out3: now also J7.T
- net VREF: now reaches U2.13 (-)
- net VREF: now also U2.14, U2.5 (+)
- net Out1: now reaches R1.1
- net Out1: now also J4.T
- new net: D2.2 (A), J6.T
- new net: D2.1 (K), R22.2
- new net: D1.2 (A), J3.T
- new net: D1.1 (K), R21.2
- new net: D3.2 (A), J9.T
- new net: D3.1 (K), R23.2
Other:
- note added: "Buffer the artificial ground"
- note added: "CV Inputs to Vactrol"
- note added: "Double Footprints Just Place One"
- note added: "Four Corners"
- note added: "Input"
- note added: "Output"
- note added: "Power Conditioning"
- company: (none) -> Karltron
- title: (none) -> Synthcard:Karltron
- moved on the sheet: C1, C2, C3, C4, C5, C6, H1, H2, H3, H4, R1, R10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

Commit message: halfway done
Parts:
- removed R6: 100K, Resistor_THT:R_Axial_DIN0207_L6.3mm_D2.5mm_P10.16mm_Horizontal, symbol Device:R
- removed R9: 10K, Resistor_THT:R_Axial_DIN0207_L6.3mm_D2.5mm_P10.16mm_Horizontal, symbol Device:R
- added R24: 100K, Resistor_THT:R_Axial_DIN0207_L6.3mm_D2.5mm_P10.16mm_Horizontal, symbol Device:R
- added R25, R26: 1M, Resistor_THT:R_Axial_DIN0207_L6.3mm_D2.5mm_P10.16mm_Horizontal, symbol Device:R
- added R6, R9: LDR, Resistor_THT:R_Axial_DIN0204_L3.6mm_D1.6mm_P5.08mm_Horizontal, symbol Device:R_Small
- J3, J4, J5, J6, J7, J8, J9: symbol Connector:AudioJack2 -> Connector_Generic:Conn_01x02
- R11: footprint Resistor_THT:R_Axial_DIN0207_L6.3mm_D2.5mm_P10.16mm_Horizontal -> Resistor_THT:R_Axial_DIN0204_L3.6mm_D1.6mm_P5.08mm_Horizontal; symbol Device:R -> Device:R_Small
- R16: value 1M -> 10K
- R17: value 100K -> 10K
- R18: value 1M -> 100K
- R4, R8: value LDR -> 1K
- R5: value 10K -> 1K
Connections:
- net GND: now also J3.2 (Pin_2), J4.2 (Pin_2), J5.2 (Pin_2), J6.2 (Pin_2), J7.2 (Pin_2), J8.2 (Pin_2), J9.2 (Pin_2); no longer J3.S, J4.S, J5.S, J6.S, J7.S, J8.S, J9.S
- net Out1: now also J4.1 (Pin_1), R20.1, U1.8; no longer J4.T
- net Out2: now also J5.1 (Pin_1), U1.14, R25.1; no longer J5.T
- net Out3: now also J7.1 (Pin_1), U2.8, R26.1; no longer J7.T
- net Out4: now also J8.1 (Pin_1); no longer J8.T
- net VREF: now also C1.2, C2.2, C3.2, R12.1, R16.1, R17.1, U1.10 (+), U1.12 (+), U2.10 (+)
- net at RV2.1: now also R5.2, RV2.2, RV6.1, RV6.2, R6.1
- net at RV2.3: now also R10.2, RV6.3, U1.7, R6.2
- net at D2.2 (A): now also J6.1 (Pin_1); no longer J6.T
- net at U1.13 (-): now also R18.1, R25.2
- net at RV5.1: now also R11.1, R4.2, RV1.1, RV1.2, RV5.2
- net at RV5.3: now also R11.2, R19.2, RV1.3, U1.1
- net Tri1: now reaches U1.2 (-)
- net Tri1: now also C1.1, R13.2, R4.1
- net at U1.3 (+): now also R12.2, R19.1
- net Tri3: now reaches R8.1
- net Tri3: now also C3.1, U2.2 (-), R24.2
- net at R8.2: now also RV3.1, RV3.2, RV7.1, RV7.2, R9.1
- net at R13.1: now also R20.2, U1.9 (-)
- net at D1.2 (A): now also J3.1 (Pin_1); no longer J3.T
- net Tri2: now reaches R18.2
- net Tri2: now also C2.1, R5.1, U1.6 (-)
- net at U2.1: now also R15.2, RV3.3, RV7.3, R9.2
- net at U2.3 (+): now also R15.1, R17.2
- net at D3.2 (A): now also J9.1 (Pin_1); no longer J9.T
- net at R16.2: now also R10.1, U1.5 (+)
- net at U2.9 (-): now also R24.1, R26.2
Other:
- note added: "Buffer & Scale"
- note added: "Relaxation Osc"
- moved on the sheet: C1, D1, D2, D3, R11, R12, R13, R19, R20, R21, R22, R23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
