File: sc_karltron/sc_karltron.kicad_sch (KiCad schematic)
At the start: 58 parts, among them J1 Conn_01x02, J2 Conn_01x02, J3 In1, J4 Out1, J5 Out2, J6 In2, J7 Out3, J8 Out4, J9 In3, U1 TL074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

Commit message: adding notes
Other:
- note added: "schem untested developed in circuit.js and breadboard but physically not yet checked"
Changed lines of the file:
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@@
   (title_block
     (title "Synthcard:Karltron")
-    (date "2023-01-16")
-    (rev "0.2")
+    (date "2023-01-19")
+    (rev "1.0")
     (company "Karltron")
     (comment 1 "karl.stamm@gmail.com")
@@
   )
   (text "Output" (at 159.385 193.04 0)
+    (effects (font (size 1.27 1.27)) (justify left bottom))
+  )
+  (text "schem untested\ndeveloped in circuit.js and breadboard\nbut physically not yet checked"
+    (at 133.35 20.955 0)
     (effects (font (size 1.27 1.27)) (justify left bottom))
   )
@@
   (symbol (lib_id "power:GND") (at 102.87 104.775 0) (unit 1)
     (in_bom yes) (on_board yes) (fields_autoplaced)
-    (property "Reference" "#PWR?" (id 0) (at 102.87 111.125 0)
+    (property "Reference" "#PWR0117" (id 0) (at 102.87 111.125 0)
       (effects (font (size 1.27 1.27)) hide)
     )
@@
   (symbol (lib_id "power:GND") (at 51.435 104.775 0) (unit 1)
     (in_bom yes) (on_board yes) (fields_autoplaced)
-    (property "Reference" "#PWR?" (id 0) (at 51.435 111.125 0)
+    (property "Reference" "#PWR0118" (id 0) (at 51.435 111.125 0)
       (effects (font (size 1.27 1.27)) hide)
     )
@@
   (symbol (lib_id "power:GND") (at 153.67 104.775 0) (unit 1)
     (in_bom yes) (on_board yes) (fields_autoplaced)
-    (property "Reference" "#PWR?" (id 0) (at 153.67 111.125 0)
+    (property "Reference" "#PWR0116" (id 0) (at 153.67 111.125 0)
       (effects (font (size 1.27 1.27)) hide)
     )
@@
       (reference "#PWR0115") (unit 1) (value "GND") (footprint "")
     )
+    (path "/38e51621-c715-4774-a18d-d6fd4aff0936"
+      (reference "#PWR0116") (unit 1) (value "GND") (footprint "")
+    )
     (path "/2c8d7a4d-c931-46a5-bcb4-c0425dc9651e"
-      (reference "#PWR?") (unit 1) (value "GND") (footprint "")
+      (reference "#PWR0117") (unit 1) (value "GND") (footprint "")
     )
     (path "/384a375b-aec0-438e-9fd5-e782aa4ca86b"
-      (reference "#PWR?") (unit 1) (value "GND") (footprint "")
-    )
-    (path "/38e51621-c715-4774-a18d-d6fd4aff0936"
-      (reference "#PWR?") (unit 1) (value "GND") (footprint "")
+      (reference "#PWR0118") (unit 1) (value "GND") (footprint "")
     )
     (path "/99c46d36-c18a-403b-9df8-c7eabf953fd1"

Commit message: after build
Other:
- note added: "Timing Capacitors are your choice 1u gives 40Hz to 4kHz 2.2uF gives 15Hz to 1.5kHz 10uF gives 4Hz to 240Hz mix it up tested w/ tl074 on 5v and 12v"
- note added: "tested working developed in circuit.js and breadboard"
- note added: "warning , no reverse polarity protection here"
- note removed: "schem untested developed in circuit.js and breadboard but physically not yet checked"
Changed lines of the file:
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@@
     (effects (font (size 1.27 1.27)) (justify left bottom))
   )
-  (text "schem untested\ndeveloped in circuit.js and breadboard\nbut physically not yet checked"
+  (text "tested working\ndeveloped in circuit.js and breadboard\n"
     (at 133.35 20.955 0)
     (effects (font (size 1.27 1.27)) (justify left bottom))
@@
     (effects (font (size 1.27 1.27)) (justify left bottom))
   )
+  (text "Timing Capacitors are your choice\n1u gives 40Hz to 4kHz\n2.2uF gives 15Hz to 1.5kHz\n10uF gives 4Hz to 240Hz\nmix it up\ntested w/ tl074 on 5v and 12v"
+    (at 197.485 95.885 0)
+    (effects (font (size 1.27 1.27)) (justify left bottom))
+  )
   (text "Buffer & Scale" (at 42.545 137.795 180)
     (effects (font (size 1.27 1.27)) (justify right bottom))
   )
+  (text "warning , no reverse polarity protection here" (at 118.745 172.72 0)
+    (effects (font (size 1.27 1.27)) (justify left bottom))
+  )
   (text "Relaxation Osc" (at 40.005 99.695 180)
