File: sc_karltron/sc_karltron.kicad_pcb (KiCad board)
At the start: 2 copper layers, 88.6 x 50.6 mm, 59 parts, among them J1 Conn_01x02, J2 Conn_01x02, J3 In1, J4 Out1, J5 Out2, J6 In2, J7 Out3, J8 Out4, J9 In3, U1 TL074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

Commit message: printing
first test - unproven
Parts:
- moved J3 0.10 mm to (110.2, 69.3)
Other:
- board text added: "+ G"
- board text added: "LDR are sensitive, isolate with black tape"
- board text added: "~1K"
- board text removed: "+ 0"
Changed lines of the file:
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@@
       (outputformat 1)
       (mirror false)
-      (drillshape 1)
+      (drillshape 0)
       (scaleselection 1)
-      (outputdirectory "")
+      (outputdirectory "gbr")
     )
   )
@@
   )
   (footprint "Connector_PinHeader_2.54mm:PinHeader_1x02_P2.54mm_Vertical" (layer "F.Cu")
-    (at 110.175 69.2 -90)
+    (at 110.175 69.3 -90)
     (descr "Through hole straight pin header, 1x02, 2.54mm pitch, single row")
     (tags "Through hole pin header THT 1x02 2.54mm single row")
@@
   (gr_arc (start 185.5 67.4) (mid 187.621319 68.278681) (end 188.5 70.4) (layer "Edge.Cuts") (width 0.1))
   (gr_line (start 99.9 115) (end 99.9 70.4) (layer "Edge.Cuts") (width 0.1))
-  (gr_text "this card\nbecomes a\n    real\n    VCO/LFO" (at 184 84.1) (layer "B.SilkS")
+  (gr_text " this card\nbecomes a\n    real\n   VCO/LFO" (at 183.8 84.2) (layer "B.SilkS")
     (effects (font (size 1.5 1.5) (thickness 0.2)) (justify left mirror))
   )
@@
     (effects (font (size 1 1) (thickness 0.15)))
   )
-  (gr_text "+\n0" (at 187.6 85.2) (layer "F.SilkS")
-    (effects (font (size 1.5 1.5) (thickness 0.2)))
-  )
   (gr_text "B100K" (at 175.5 100.6) (layer "F.SilkS")
     (effects (font (size 1 1) (thickness 0.15)))
@@
     (effects (font (size 1.5 1.5) (thickness 0.2)))
   )
-  (gr_text "+\n0" (at 187.7 92.8) (layer "F.SilkS")
-    (effects (font (size 1.5 1.5) (thickness 0.2)))
+  (gr_text "+\nG" (at 187.5 92.8) (layer "F.SilkS")
+    (effects (font (size 1.5 1.4) (thickness 0.2)))
   )
   (gr_text "out\n1" (at 184.2 74.2 90) (layer "F.SilkS")
@@
     (effects (font (size 1.25 1.25) (thickness 0.17)))
   )
-  (gr_text "+\n0" (at 187.7 100.5) (layer "F.SilkS")
-    (effects (font (size 1.5 1.5) (thickness 0.2)))
+  (gr_text "+\nG" (at 187.5 77.7) (layer "F.SilkS")
+    (effects (font (size 1.5 1.4) (thickness 0.2)))
   )
   (gr_text "-" (at 153.1 92.3) (layer "F.SilkS")
     (effects (font (size 0.5 0.5) (thickness 0.125)))
   )
+  (gr_text "~1K" (at 112.5 80.2 90) (layer "F.SilkS")
+    (effects (font (size 1 1) (thickness 0.15)))
+  )
   (gr_text "Karltron\nTriple VCO/LFO\nSynthcard" (at 144.5 86.9) (layer "F.SilkS")
     (effects (font (size 1.7 1.7) (thickness 0.25)))
   )
-  (gr_text "1" (at 112.5 69.1) (layer "F.SilkS")
+  (gr_text "LDR are sensitive, isolate with black tape" (at 117.5 87.1) (layer "F.SilkS")
+    (effects (font (size 1 1) (thickness 0.15)))
+  )
+  (gr_text "1" (at 112.5 69.3) (layer "F.SilkS")
     (effects (font (size 1.25 1.25) (thickness 0.17)))
   )
@@
     (effects (font (size 1.25 1.25) (thickness 0.17)))
   )
-  (gr_text "+\n0" (at 187.6 77.6) (layer "F.SilkS")
-    (effects (font (size 1.5 1.5) (thickness 0.2)))
-  )
   (gr_text "B100K" (at 177.3 72.4) (layer "F.SilkS")
     (effects (font (size 1 1) (thickness 0.15)))
@@
     (effects (font (size 1.25 1.25) (thickness 0.17)))
   )
-  (gr_text "2" (at 122.6 69.2) (layer "F.SilkS")
+  (gr_text "2" (at 122.6 69.3) (layer "F.SilkS")
     (effects (font (size 1.25 1.25) (thickness 0.17)))
   )
@@
     (effects (font (size 1 1) (thickness 0.15)))
   )
+  (gr_text "+\nG" (at 187.5 100.5) (layer "F.SilkS")
+    (effects (font (size 1.5 1.4) (thickness 0.2)))
+  )
   (gr_text "2" (at 165.7 70) (layer "F.SilkS")
     (effects (font (size 1.25 1.25) (thickness 0.17)))
@@
     (effects (font (size 1.5 1.5) (thickness 0.2)))
   )
-  (gr_text "3" (at 133.8 69.2) (layer "F.SilkS")
+  (gr_text "3" (at 133.8 69.3) (layer "F.SilkS")
     (effects (font (size 1.25 1.25) (thickness 0.17)))
   )
@@
     (effects (font (size 1.5 1.5) (thickness 0.2)))
   )
+  (gr_text "+\nG" (at 187.5 85.2) (layer "F.SilkS")
+    (effects (font (size 1.5 1.4) (thickness 0.2)))
+  )
   (gr_text "file not tested physically\ni still need to order one and build it \n  before i can guarantee this board is good" (at 144.1 49.7) (layer "Cmts.User")

Commit message: after build
Other:
- board text added: "tested working RLED 1K is good for 5Vcc but weak at 12Vcc Caps 1u to 10u give lfo to vco range"
- board text removed: "file not tested physically i still need to order one and build it before i can guarantee this board is good"
Changed lines of the file:
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@@
     (property "Sheetfile" "sc_karltron.kicad_sch")
     (property "Sheetname" "")
-    (attr exclude_from_pos_files)
+    (attr exclude_from_bom)
     (fp_text reference "H4" (at 0 -4.2) (layer "F.SilkS") hide
       (effects (font (size 1 1) (thickness 0.15)))
@@
     (property "Sheetfile" "sc_karltron.kicad_sch")
     (property "Sheetname" "")
-    (attr exclude_from_pos_files)
+    (attr exclude_from_bom)
     (fp_text reference "H2" (at 0 -4.2) (layer "F.SilkS") hide
       (effects (font (size 1 1) (thickness 0.15)))
@@
     (property "Sheetfile" "sc_karltron.kicad_sch")
     (property "Sheetname" "")
-    (attr exclude_from_pos_files)
+    (attr exclude_from_bom)
     (fp_text reference "H1" (at 0 -4.2) (layer "F.SilkS") hide
       (effects (font (size 1 1) (thickness 0.15)))
@@
     (property "Sheetfile" "sc_karltron.kicad_sch")
     (property "Sheetname" "")
-    (attr exclude_from_pos_files)
+    (attr exclude_from_bom)
     (fp_text reference "H3" (at 0 -4.2) (layer "F.SilkS") hide
       (effects (font (size 1 1) (thickness 0.15)))
@@
     (effects (font (size 2 2) (thickness 0.25)) (justify right mirror))
   )
+  (gr_text "+\n-" (at 187 108.7) (layer "B.SilkS")
+    (effects (font (size 1.5 1.5) (thickness 0.2)) (justify mirror))
+  )
   (gr_text "Don't be scared\nto try it!" (at 110.3 99.5) (layer "B.SilkS")
     (effects (font (size 1.5 1.5) (thickness 0.2)) (justify mirror))
@@
     (effects (font (size 1.75 1.75) (thickness 0.25)) (justify right mirror))
   )
+  (gr_text "+\n-" (at 101.5 108.7) (layer "B.SilkS")
+    (effects (font (size 1.5 1.5) (thickness 0.2)) (justify mirror))
+  )
   (gr_text "instagram.com/karltronsynth" (at 126.1 113.7) (layer "B.SilkS")
     (effects (font (size 1.5 1.5) (thickness 0.2)) (justify mirror))
@@
     (effects (font (size 1.5 1.4) (thickness 0.2)))
   )
-  (gr_text "file not tested physically\ni still need to order one and build it \n  before i can guarantee this board is good" (at 144.1 49.7) (layer "Cmts.User")
+  (gr_text "tested working\nRLED 1K is good for 5Vcc but weak at 12Vcc\nCaps 1u to 10u give lfo to vco range" (at 144.1 49.7) (layer "Cmts.User")
     (effects (font (size 2 2) (thickness 0.2)))
   )
