File: sc_ex1/sc_ex1.kicad_pcb (KiCad board)
At the start: 2 copper layers, 88.6 x 50.6 mm, 6 parts, among them J1 Conn_01x02, J2 Conn_01x02

Commit message: tweaks, bugfix
moved measurements and courtyards
Other:
- board text added: "The +V power rail continues on top and bottom of the board this is not necessary, if you want the space, remove one side. Connect the power pins to daisy-chain synthcards"
